File: hardware/schematics/microloop.kicad_sch (KiCad schematic)
At the start: 31 parts, among them J1 Stereo Input, J2 Stereo Output, SW1 Rotary Encoder + Button, SW2 Rotary Encoder + Button, SW3 Rotary Encoder + Button, SW4 Rotary Encoder + Button, SW5 Preset Button, SW6 Preset Button, SW7 Preset Button, SW8 Preset Button, U1 Teensy 4.1, U2 Teensy Audio Shield (Rev D), U3 Adafruit MIDI Featherwing, U5 MCP23017, U6 OLED 128×64, U7 Adafruit NeoKey 1x4

Commit message: finalized schematic, added bom
Parts:
- J1: value Stereo Input -> Stereo Line In
- J2: value Stereo Output -> Stereo Line Out
- U1: symbol teensy:Teensy4.1 -> microloop_symbols:Teensy4.1
- U2: symbol teensy4.0_audioshield_revd:Teensy4.0_AudioShield_REVD -> microloop_symbols:Teensy4.0_AudioShield_REVD
- U3: symbol new:midi -> microloop_symbols:midi
- U6: value OLED 128×64 -> SSD1306 OLED; symbol new:oled -> microloop_symbols:oled
- U7: symbol new:neokey -> microloop_symbols:neokey
Connections:
- net +3.3V: no longer U3.2 (3.3V), U6.2 (VCC), U7.1 (VIN)
- net GND: now also SW1.C, SW2.C, SW3.C, SW4.C; no longer U3.4 (GND), U6.1 (GND), U7.3 (GND)
- net NeoKey_INT: no longer U7.6 (INT)
- net Serial8_RX: no longer U3.14 (RX)
- net Serial8_TX: no longer U3.15 (TX)
- net Wire1_CLK: no longer U6.3 (SCL)
- net Wire1_SDA: no longer U6.4 (SDA)
- net Wire2_CLK: no longer U7.4 (CLK)
- net Wire2_SDA: no longer U7.5 (SDA)
- net PRST_LED_2: now reaches R4.2
- net PRST_LED_2: now also U1.22 (30_CRX3)
- net IND_LED_G: now reaches R7.2
- net IND_LED_G: now also U1.28 (36_CS)
- net BEAT_LED: now reaches R1.2
- net BEAT_LED: now also U1.30 (38_CS1_IN1)
- net PRST_LED_3: now reaches R3.2
- net PRST_LED_3: now also U1.23 (31_CTX3)
- net IND_LED_R: now reaches U1.20 (28_RX7)
- net IND_LED_R: now also R6.2
- net PRST_LED_1: now reaches U1.21 (29_TX7)
- net PRST_LED_1: now also R5.2
- net PRST_LED_4: now reaches U1.24 (32_OUT1B)
- net PRST_LED_4: now also R2.2
- net IND_LED_B: now reaches U1.29 (37_CS)
- net IND_LED_B: now also R8.2
- net LINE_IN_R: now reaches J1.R, U2.34 (LINE_IN_R)
- net LINE_IN_GND: now reaches J1.S, U2.36 (LINE_IN_R_GND)
- net LINE_IN_L: now reaches J1.T, U2.35 (LINE_IN_L)
- net ENC_A_3: now reaches SW3.A
- net ENC_A_3: now also U5.4 (GPB3)
- net ENC_B_3: now reaches SW3.B
- net ENC_B_3: now also U5.5 (GPB4)
- net ENC_SW_3: now reaches SW3.S1
- net ENC_SW_3: now also U5.6 (GPB5)
- net ENC_A_4: now reaches SW4.A
- net ENC_A_4: now also U5.28 (GPA7)
- net ENC_B_4: now reaches SW4.B
- net ENC_B_4: now also U5.27 (GPA6)
- net ENC_SW_4: now reaches SW4.S1
- net ENC_SW_4: now also U5.26 (GPA5)
- net ENC_A_1: now reaches SW1.A
- net ENC_A_1: now also U5.25 (GPA4)
- net ENC_B_1: now reaches SW1.B
- net ENC_B_1: now also U5.24 (GPA3)
- net ENC_SW_1: now reaches SW1.S1
- net ENC_SW_1: now also U5.23 (GPA2)
- net LINE_OUT_L: now reaches J2.T, U2.31 (LINE_OUT_L)
- net LINE_OUT_GND: now reaches J2.S, U2.32 (LINE_OUT_GND)
- net LINE_OUT_R: now reaches J2.R, U2.33 (LINE_OUT_R)
- net ENC_A_2: now reaches U5.1 (GPB0)
- net ENC_A_2: now also SW2.A
- net ENC_B_2: now reaches U5.2 (GPB1)
- net ENC_B_2: now also SW2.B
- net PRST_SW_2: now reaches U5.21 (GPA0)
- net PRST_SW_2: now also SW7.2
- net PRST_SW_1: now reaches U5.22 (GPA1)
- net PRST_SW_1: now also SW8.2
- net ENC_SW_2: now reaches U5.3 (GPB2)
- net ENC_SW_2: now also SW2.S1
- net PRST_SW_3: now reaches U5.7 (GPB6)
- net PRST_SW_3: now also SW6.2
- net PRST_SW_4: now reaches U5.8 (GPB7)
- net PRST_SW_4: now also SW5.2
- no-connect marks 54 -> 58
Other:
- note added: "APS6404L 8 MB PSRAM chip soldered on underside pads, between pins 31-32 and 33-34."
- note added: "Place decoupling capacitor as close as possible to MCP23017 VDD and VSS pins."
- title: (none) -> MicroLoop
- moved on the sheet: C1, D1, D2, D3, D4, D5, D6, J1, R1, R2, R3, R4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

Commit message: added sd card to bom + schematic
Other:
- note added: "microSD card goes in Teensy's port, NOT the Audio Adapter's."
Changed lines of the file:
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@@
+		)
+	)
+	(text "microSD card goes in Teensy's port, NOT the Audio Adapter's."
+		(exclude_from_sim no)
+		(at 270.764 146.05 0)
+		(effects
+			(font
+				(size 1.27 1.27)
+			)
 		)
 	)
 	(text "APS6404L 8 MB PSRAM chip soldered on underside pads,\nbetween pins 31-32 and 33-34."
 		(exclude_from_sim no)
-		(at 270.51 148.844 0)
+		(at 270.51 151.638 0)
 		(effects
 			(font

Commit message: cleaned up presets, updated hardware
Parts:
- R7, R8: value 100R -> 330R
Connections:
- net PRST_SW_1: now also U1.32 (40_A16); no longer U5.22 (GPA1)
- net PRST_SW_2: now also U1.33 (41_A17); no longer U5.21 (GPA0)
- net PRST_SW_3: now also U1.19 (27_A13_SCK1); no longer U5.7 (GPB6)
- net PRST_SW_4: now also U1.18 (26_A12_MOSI1); no longer U5.8 (GPB7)
Changed lines of the file:
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@@
 	)
 	(no_connect
-		(at 242.57 96.52)
-	)
-	(no_connect
 		(at 242.57 116.84)
 	)
@@
 	)
 	(no_connect
+		(at 372.11 184.15)
+	)
+	(no_connect
 		(at 46.99 72.39)
 	)
@@
 	)
 	(no_connect
-		(at 298.45 91.44)
+		(at 372.11 194.31)
+	)
+	(no_connect
+		(at 372.11 191.77)
 	)
 	(no_connect
@@
 	)
 	(no_connect
-		(at 298.45 93.98)
-	)
-	(no_connect
 		(at 46.99 67.31)
 	)
@@
 	)
 	(no_connect
-		(at 242.57 99.06)
-	)
-	(no_connect
 		(at 266.7 140.97)
 	)
@@
 	)
 	(no_connect
+		(at 372.11 186.69)
+	)
+	(no_connect
 		(at 392.43 60.96)
 	)
@@
 	(wire
 		(pts
+			(xy 231.14 96.52) (xy 242.57 96.52)
+		)
+		(stroke
+			(width 0)
+			(type default)
+		)
+	)
+	(wire
+		(pts
 			(xy 298.45 104.14) (xy 308.61 104.14)
 		)
@@
 	(wire
 		(pts
+			(xy 298.45 91.44) (xy 309.88 91.44)
+		)
+		(stroke
+			(width 0)
+			(type default)
+		)
+	)
+	(wire
+		(pts
 			(xy 96.52 137.16) (xy 92.71 137.16)
 		)
@@
 	(wire
 		(pts
-			(xy 372.11 194.31) (xy 383.54 194.31)
-		)
-		(stroke
-			(width 0)
-			(type default)
-		)
-	)
-	(wire
-		(pts
 			(xy 50.8 237.49) (xy 59.69 237.49)
 		)
@@
 	(wire
 		(pts
-			(xy 298.45 88.9) (xy 311.15 88.9)
+			(xy 298.45 88.9) (xy 314.96 88.9)
 		)
 		(stroke
@@
 	(wire
 		(pts
-			(xy 372.11 184.15) (xy 383.54 184.15)
+			(xy 233.68 53.34) (xy 242.57 53.34)
 		)
 		(stroke
@@
 	(wire
 		(pts
-			(xy 233.68 53.34) (xy 242.57 53.34)
+			(xy 298.45 93.98) (xy 309.88 93.98)
 		)
 		(stroke
@@
 	(wire
 		(pts
-			(xy 372.11 191.77) (xy 383.54 191.77)
+			(xy 205.74 198.12) (xy 207.01 198.12)
 		)
 		(stroke
@@
 	(wire
 		(pts
-			(xy 205.74 198.12) (xy 207.01 198.12)
+			(xy 331.47 52.07) (xy 336.55 52.07)
 		)
 		(stroke
@@
 	(wire
 		(pts
-			(xy 331.47 52.07) (xy 336.55 52.07)
+			(xy 298.45 55.88) (xy 307.34 55.88)
 		)
 		(stroke
@@
 	(wire
 		(pts
-			(xy 298.45 55.88) (xy 307.34 55.88)
+			(xy 193.04 203.2) (xy 207.01 203.2)
 		)
 		(stroke
@@
 	(wire
 		(pts
-			(xy 193.04 203.2) (xy 207.01 203.2)
+			(xy 260.35 224.79) (xy 271.78 224.79)
 		)
 		(stroke
@@
 	(wire
 		(pts
-			(xy 260.35 224.79) (xy 271.78 224.79)
+			(xy 231.14 99.06) (xy 242.57 99.06)
 		)
 		(stroke
@@
 	(wire
 		(pts
-			(xy 372.11 186.69) (xy 383.54 186.69)
-		)
-		(stroke
-			(width 0)
-			(type default)
-		)
-	)
-	(wire
-		(pts
 			(xy 298.45 76.2) (xy 308.61 76.2)
 		)
@@
 		)
 	)
+	(label "PRST_SW_4"
+		(at 231.14 96.52 0)
+		(effects
+			(font
+				(size 1.27 1.27)
+			)
+			(justify left bottom)
+		)
+	)
 	(label "Wire1_CLK"
 		(at 172.72 87.63 0)
@@
 	)
 	(label "PRST_SW_2"
-		(at 372.11 191.77 0)
+		(at 298.45 91.44 0)
 		(effects
 			(font
@@
 		)
 	)
-	(label "PRST_LED_1"
-		(at 231.14 104.14 0)
+	(label "PRST_SW_3"
+		(at 231.14 99.06 0)
 		(effects
 			(font
@@
 		)
 	)
-	(label "ENC_SW_3"
-		(at 76.2 232.41 0)
+	(label "PRST_LED_1"
+		(at 231.14 104.14 0)
 		(effects
 			(font
@@
 		)
 	)
-	(label "Wire1_SDA"
-		(at 298.45 76.2 0)
+	(label "ENC_SW_3"
+		(at 76.2 232.41 0)
 		(effects
 			(font
@@
 		)
 	)
-	(label "PRST_SW_3"
-		(at 372.11 184.15 0)
+	(label "Wire1_SDA"
+		(at 298.45 76.2 0)
 		(effects
 			(font
@@
 		)
 	)
+	(label "PRST_SW_1"
+		(at 298.45 93.98 0)
+		(effects
+			(font
+				(size 1.27 1.27)
+			)
+			(justify left bottom)
+		)
+	)
 	(label "ENC_B_4"
 		(at 119.38 237.49 0)
@@
 		)
 	)
-	(label "PRST_SW_4"
-		(at 372.11 186.69 0)
-		(effects
-			(font
-				(size 1.27 1.27)
-			)
-			(justify left bottom)
-		)
-	)
 	(label "AA_22"
 		(at 392.43 118.11 0)
@@
 		)
 	)
-	(label "PRST_SW_1"
-		(at 372.11 194.31 0)
-		(effects
-			(font
-				(size 1.27 1.27)
-			)
-			(justify left bottom)
-		)
-	)
 	(label "PRST_LED_3"
 		(at 231.14 109.22 0)
@@
 			)
 		)
-		(property "Value" "100R"
+		(property "Value" "330R"
 			(at 119.38 88.8999 90)
 			(effects
@@
 			)
 		)
-		(property "Value" "100R"
+		(property "Value" "330R"
 			(at 119.38 99.0599 90)
 			(effects
@@
 	(symbol
 		(lib_id "power:GND")
-		(at 311.15 88.9 0)
+		(at 314.96 88.9 0)
 		(unit 1)
 		(exclude_from_sim no)
@@
 		(on_board yes)
 		(dnp no)
-		(fields_autoplaced yes)
 		(property "Reference" "#PWR01"
-			(at 311.15 95.25 0)
+			(at 314.96 95.25 0)
 			(effects
 				(font
@@
 		)
 		(property "Value" "GND"
-			(at 311.15 93.98 0)
+			(at 314.96 93.98 0)
 			(effects
 				(font
@@
 		)
 		(property "Footprint" ""
-			(at 311.15 88.9 0)
+			(at 314.96 88.9 0)
 			(effects
 				(font
@@
 		)
 		(property "Datasheet" ""
-			(at 311.15 88.9 0)
+			(at 314.96 88.9 0)
 			(effects
 				(font
@@
 		)
 		(property "Description" "Power symbol creates a global label with name \"GND\" , ground"
-			(at 311.15 88.9 0)
+			(at 314.96 88.9 0)
 			(effects
 				(font

Commit message: added libraries, changed README
Connections:
- net +3.3V: now also U3.2 (3.3V), U6.2 (VCC), U7.1 (VIN)
- net GND: now also U3.4 (GND), U6.1 (GND), U7.3 (GND)
- net NeoKey_INT: now also U7.6 (INT)
- net Serial8_RX: now also U3.14 (RX)
- net Serial8_TX: now also U3.15 (TX)
- net Wire1_CLK: now also U6.3 (SCL)
- net Wire1_SDA: now also U6.4 (SDA)
- net Wire2_CLK: now also U7.4 (CLK)
- net Wire2_SDA: now also U7.5 (SDA)
Other:
- moved on the sheet: U6, U7

Commit message: pcb wip 2/18
Parts:
- removed U3: Adafruit MIDI Featherwing, symbol microloop_symbols:midi
- added D7: 1N4148, Diode_THT:D_DO-35_SOD27_P7.62mm_Horizontal, symbol Diode:1N4148
- added J4: MIDI DIN-5, symbol Connector:DIN-5_180degree
- added R10: 470R, symbol Device:R_US
- added R9: 220R, symbol Device:R_US
- added U4: H11L1SM, H11L1SM:IC_H11L1SM, symbol H11L1SM:H11L1SM
Connections:
- net AA_GND2 is gone; now on net GND: U1.1 (GND), U1.47 (GND), U2.1 (GND), U2.29 (GND)
- net +3.3V: now also R10.1, U4.6
- net GND: now also U4.5
- net Serial8_RX: now also R10.2, U4.4
- net AA_10 renamed AA_SDCS
- net AA_11 renamed AA_MOSI
- net AA_12 renamed AA_MISO
- net AA_13 renamed AA_SCK
- net AA_15 renamed AA_VOL
- net AA_20 renamed AA_LRCLK
- net AA_21 renamed AA_BCLK
- net AA_23 renamed AA_MCLK
- net AA_5V renamed +5V
- net AA_6 renamed AA_MEMCS
- net AA_7 renamed AA_DIN
- net AA_8 renamed AA_DOUT
- net Serial8_TX: no longer names the net of U1.27 (35_TX8)
- new net: D7.1 (K), R9.2, U4.1
- new net: D7.2 (A), J4.5, U4.2
- new net: J4.4, R9.1
- no-connect marks 58 -> 38
Other:
- note added: "AA_'NUM' means unused pins that are still connected to the Audio Adapter. The Teensy and Audio Adapter board should be mounted directly on top of each other, per PJRC guidelines."
- note removed: "'AA' means Audio Adapter pins that aren't used for anything else. The Teensy and Audio Adapter board should be mounted directly on top of each other, per PJRC guidelines."
- moved on the sheet: D1, D2, R1, R6, R7, R8, U6

Commit message: updated keys+leds
Parts:
- added D10, D11, D12, D13, D14, D15, D16, D17, D18, D19, D8, D9: SK6812MINI, LED_SMD:LED_SK6812MINI_PLCC4_3.5x3.5mm_P1.75mm, symbol LED:SK6812MINI
- added SW10, SW11, SW12, SW13, SW14, SW15, SW16, SW17: Preset Button, symbol Switch:SW_Push
- added U8: SN74AHCT1G125DBVR, symbol microloop_symbols:SN74
- C1: footprint (none) -> Capacitor_SMD:C_0805_2012Metric_Pad1.18x1.45mm_HandSolder
- R1, R10, R2, R3, R4, R5, R6, R7, R8, R9: footprint (none) -> Resistor_SMD:R_0805_2012Metric_Pad1.20x1.40mm_HandSolder
- U5: value MCP23017 -> Encoders - MCP23017
Connections:
- net AA_0 is gone; now on net PRST_SW_1: U1.2 (0_RX1_CRX2_CS1), U2.2 (0_RX1_CRX2_CS1)
- net AA_1 is gone; now on net PRST_SW_2: U1.3 (1_TX1_CTX2_MISO1), U2.3 (1_TX1_CTX2_MISO1)
- net AA_2 is gone; now on net PRST_SW_3: U1.4 (2_OUT2), U2.4 (2_OUT2)
- net AA_3 is gone; now on net PRST_SW_4: U1.5 (3_LRCLK2), U2.5 (3_LRCLK2)
- net +5V: now also D10.4 (VDD), D11.4 (VDD), D12.4 (VDD), D13.4 (VDD), D14.4 (VDD), D15.4 (VDD), D16.4 (VDD), D17.4 (VDD), D18.4 (VDD), D19.4 (VDD), D8.4 (VDD), D9.4 (VDD)
- net GND: now also D10.2 (VSS), D11.2 (VSS), D12.2 (VSS), D13.2 (VSS), D14.2 (VSS), D15.2 (VSS), D16.2 (VSS), D17.2 (VSS), D18.2 (VSS), D19.2 (VSS), D8.2 (VSS), D9.2 (VSS), SW10.2, SW11.2, SW12.2, SW13.2, SW14.2, SW15.2, SW16.2, SW17.2
- net PRST_SW_1: now also SW10.1; no longer U1.32 (40_A16)
- net PRST_SW_2: now also SW11.1; no longer U1.33 (41_A17)
- net PRST_SW_3: now also SW12.1; no longer U1.19 (27_A13_SCK1)
- net PRST_SW_4: now also SW13.1; no longer U1.18 (26_A12_MOSI1)
- net AA_22 renamed PRST_SW_8
- net PRST_SW_8: now also SW17.1
- net AA_4 renamed PRST_SW_5
- net PRST_SW_5: now also SW14.1
- net AA_5 renamed PRST_SW_6
- net PRST_SW_6: now also SW15.1
- net AA_9 renamed PRST_SW_7
- net PRST_SW_7: now also SW16.1
- new net: D12.1 (DOUT), D13.3 (DIN)
- new net: D12.3 (DIN), D8.3 (DIN)
- new net: D15.1 (DOUT), D17.3 (DIN)
- new net: D14.1 (DOUT), D15.3 (DIN)
- new net: D10.1 (DOUT), D11.3 (DIN)
- new net: D10.3 (DIN), D9.1 (DOUT)
- new net: D11.1 (DOUT), D16.3 (DIN)
- new net: D16.1 (DOUT), D18.3 (DIN)
- new net: D8.1 (DOUT), D9.3 (DIN)
- new net: D13.1 (DOUT), D14.3 (DIN)
- new net: D17.1 (DOUT), D19.3 (DIN)
- no-connect marks 38 -> 39
Other:
- note added: "First in the chain gets put closest to level shifter"
- note added: "IO Expander ONLY if no pins left on teensy"
- moved on the sheet: D3, D4, D5, D6, R2, R3, R4, R5, SW1, SW2, SW3, SW4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

Commit message: switches, jacks, and smd leds
Parts:
- removed D3, D4, D5, D6: Preset LED, symbol Device:LED
- removed J1: Stereo Line In, symbol Connector_Audio:AudioJack3
- removed J2: Stereo Line Out, symbol Connector_Audio:AudioJack3
- removed R2, R3, R4, R5: 330R, Resistor_SMD:R_0805_2012Metric_Pad1.20x1.40mm_HandSolder, symbol Device:R_US
- removed SW5, SW6, SW7, SW8: Preset Button, symbol Switch:SW_Push
- removed U7: Adafruit NeoKey 1x4, symbol microloop_symbols:neokey
- added C10: 500uF, Capacitor_SMD:C_0805_2012Metric_Pad1.18x1.45mm_HandSolder, symbol Device:C
- added C11, C12, C13, C14, C15, C2, C3, C4, C5, C6, C7, C8, C9: 0.1uF, Capacitor_SMD:C_0805_2012Metric_Pad1.18x1.45mm_HandSolder, symbol Device:C
- added J1: Input L, symbol Connector_Audio:AudioJack2_Switch
- added J2: Output L, symbol Connector_Audio:AudioJack2_Switch
- added J3: Input R, symbol Connector_Audio:AudioJack2_Switch
- added J5: Output R, symbol Connector_Audio:AudioJack2_Switch
- added R11: 330R/470R, symbol Device:R_US
- added SW18, SW19, SW20, SW21: Preset Button, symbol Switch:SW_Push
- C1: value 100nF -> 0.1uF
- U8: value SN74AHCT1G125DBVR -> SN74AHCT1G125
Connections:
- net AA_14 is gone; now on net PRST_LEDS: U1.36 (14_A0_TX3_SPDIF_OUT), U2.18 (14_A0_TX3_SPDIF_OUT)
- net +5V: now also U8.5 (VCC), C10.1, C11.1, C12.1, C13.1, C14.1, C15.1, C2.1, C3.1, C4.1, C5.1, C6.1, C7.1, C8.1, C9.1
- net GND: now also U8.1 (!OE), U8.3 (GND), C10.2, C11.2, C12.2, C13.2, C14.2, C15.2, C2.2, C3.2, C4.2, C5.2, C6.2, C7.2, C8.2, C9.2, SW18.2, SW19.2, SW20.2, SW21.2
- net LINE_IN_GND: now also J1.S, J3.S
- net LINE_IN_L: now also J1.T
- net LINE_IN_R: now also J3.T
- net LINE_OUT_GND: now also J2.S, J5.S
- net LINE_OUT_L: now also J2.T
- net LINE_OUT_R: now also J5.T
- net PRST_LEDS: now reaches U8.2 (A)
- net at U8.4 (Y): now also R11.2
- net at D8.3 (DIN): now also R11.1; no longer D12.3 (DIN)
- net LINE_OUT_DETECT: now reaches U1.32 (40_A16)
- net LINE_OUT_DETECT: now also J5.SN
- net LINE_IN_DETECT: now reaches U1.33 (41_A17)
- net LINE_IN_DETECT: now also J3.SN
- net at D17.3 (DIN): now also D16.1 (DOUT); no longer D15.1 (DOUT)
- net at D18.3 (DIN): now also D15.1 (DOUT); no longer D16.1 (DOUT)
- net at D18.1 (DOUT): now also D19.3 (DIN)
- net at D17.1 (DOUT): now also D12.3 (DIN); no longer D19.3 (DIN)
- net NeoKey_INT: no longer names the net of U1.25 (33_MCLK2)
- net PRST_LED_1 renamed PRST_SW_9
- net PRST_SW_9: now also SW18.1
- net PRST_LED_2 renamed PRST_SW_10
- net PRST_SW_10: now also SW19.1
- net PRST_LED_3 renamed PRST_SW_11
- net PRST_SW_11: now also SW20.1
- net PRST_LED_4 renamed PRST_SW_12
- net PRST_SW_12: now also SW21.1
- net Wire2_CLK: no longer names the net of U1.16 (24_A10_TX6_SCL2)
- net Wire2_SDA: no longer names the net of U1.17 (25_A11_RX6_SDA2)
- no-connect marks 39 -> 44
Other:
- note added: "Bulk cap, near where power enters first LED, across +/- terminals"
- note added: "Can move this I2C to Wire2, since we removed NeoKey"
- note added: "NEED to enable pinMode(pin, INPUT_PULLUP) for SN pins on Teensy."
- note added: "Place decoupling capacitors as close as possible from VDD/VSS or VCC/GND"
- moved on the sheet: C1, D1, D2, D8, R1, R6, R7, R8, SW1, SW10, SW11, SW12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

Commit message: added power stuff, usb-c stuff
Parts:
- removed U6: SSD1306 OLED, symbol microloop_symbols:oled
- added C16, C19: 0.1uF, Capacitor_SMD:C_0805_2012Metric_Pad1.18x1.45mm_HandSolder, symbol Device:C
- added C17: 47uF, symbol Device:C_Polarized
- added C18: C_Polarized, symbol Device:C_Polarized
- added D3: D_TVS, symbol Device:D_TVS
- added F1: Polyfuse, symbol Device:Polyfuse
- added J6: Barrel_Jack_Switch, symbol Connector:Barrel_Jack_Switch
- added J7: USB_C_Receptacle_USB2.0_14P, symbol Connector:USB_C_Receptacle_USB2.0_14P
- added SW5: SW_Push, symbol Switch:SW_Push
- added U3: SSD1309 SPI OLED, symbol microloop_symbols:SSD1309 SPI OLED
- added U6: Adafruit 1400, symbol microloop_symbols:Adafruit_1400
- added U7: Switches - MCP23017, Package_SO:SOIC-28W_7.5x17.9mm_P1.27mm, symbol Interface_Expansion:MCP23017_SO
Connections:
- net +3.3V: now also C16.1, U3.1 (GND), U7.18 (~{RESET}), U7.9 (VDD)
- net ENC_A_1: now also U5.1 (GPB0); no longer U5.25 (GPA4)
- net ENC_A_2: now also U5.4 (GPB3); no longer U5.1 (GPB0)
- net ENC_A_3: now also U5.23 (GPA2); no longer U5.4 (GPB3)
- net ENC_A_4: now also U5.26 (GPA5); no longer U5.28 (GPA7)
- net ENC_B_1: now also U5.2 (GPB1); no longer U5.24 (GPA3)
- net ENC_B_2: now also U5.5 (GPB4); no longer U5.2 (GPB1)
- net ENC_B_3: now also U5.24 (GPA3); no longer U5.5 (GPB4)
- net ENC_SW_1: now also U5.3 (GPB2); no longer U5.23 (GPA2)
- net ENC_SW_2: now also U5.6 (GPB5); no longer U5.3 (GPB2)
- net ENC_SW_3: now also U5.25 (GPA4); no longer U5.6 (GPB5)
- net ENC_SW_4: now also U5.28 (GPA7); no longer U5.26 (GPA5)
- net GND: now also C16.2, C17.2, C19.1, D3.2 (A2), J6.2, U3.2 (VCC), U6.3 (GND), U7.10 (VSS), U7.15 (A0), U7.16 (A1), U7.17 (A2)
- net IND_LED_R: now also U1.25 (33_MCLK2); no longer U1.20 (28_RX7)
- net PRST_SW_1: now also U7.1 (GPB0); no longer U1.2 (0_RX1_CRX2_CS1)
- net PRST_SW_10: now also U7.22 (GPA1); no longer U1.22 (30_CRX3)
- net PRST_SW_11: now also U7.23 (GPA2); no longer U1.23 (31_CTX3)
- net PRST_SW_12: now also U7.24 (GPA3); no longer U1.24 (32_OUT1B)
- net PRST_SW_2: now also U7.2 (GPB1); no longer U1.3 (1_TX1_CTX2_MISO1)
- net PRST_SW_3: now also U7.3 (GPB2); no longer U1.4 (2_OUT2)
- net PRST_SW_4: now also U7.4 (GPB3); no longer U1.5 (3_LRCLK2)
- net PRST_SW_5: now also U7.5 (GPB4); no longer U1.6 (4_BCLK2)
- net PRST_SW_6: now also U7.6 (GPB5); no longer U1.7 (5_IN2)
- net PRST_SW_7: now also U7.7 (GPB6); no longer U1.11 (9_OUT1C)
- net PRST_SW_8: now also U7.8 (GPB7); no longer U1.44 (22_A8_CTX1), U2.26 (22_A8_CTX1)
- net PRST_SW_9: now also U7.21 (GPA0); no longer U1.21 (29_TX7)
- net IOX_SW_CLK: now reaches U1.16 (24_A10_TX6_SCL2)
- net IOX_SW_CLK: now also U7.12 (SCK)
- net IOX_SW_SDA: now reaches U1.17 (25_A11_RX6_SDA2)
- net IOX_SW_SDA: now also U7.13 (SDA)
- net OLED_MOSI: now reaches U1.18 (26_A12_MOSI1)
- net OLED_MOSI: now also U3.4 (SDA)
- net OLED_SCK: now reaches U1.19 (27_A13_SCK1)
- net OLED_SCK: now also U3.3 (SCK)
- net MCP_INT renamed IOX_ENC_INT
- net Wire1_CLK renamed IOX_ENC_CLK
- net IOX_ENC_CLK: now also U5.12 (SCK)
- net Wire1_SDA renamed IOX_ENC_SDA
- net IOX_ENC_SDA: now also U5.13 (SDA)
- net Wire_CLK renamed AA_CLK
- net AA_CLK: no longer U5.12 (SCK)
- net Wire_SDA renamed AA_SDA
- net AA_SDA: no longer U5.13 (SDA)
- new net: C17.1, C19.2, D3.1 (A1), F1.2, U6.1 (IN)
- new net: SW5.1, U6.6 (SW2)
- new net: SW5.2, U6.5 (SW1)
- new net: J7.A1 (GND), J7.A12 (GND), J7.B1 (GND), J7.B12 (GND)
- new net: J7.A4 (VBUS), J7.A9 (VBUS), J7.B4 (VBUS), J7.B9 (VBUS)
- new net: F1.1, J6.1
- new net IOX_SW_INT: U1.20 (28_RX7), U7.20 (INTA)
- new net OLED_CS: U1.2 (0_RX1_CRX2_CS1), U3.7 (CS)
- new net OLED_DC: U1.3 (1_TX1_CTX2_MISO1), U3.6 (DC)
- new net OLED_RES: U1.44 (22_A8_CTX1), U2.26 (22_A8_CTX1), U3.5 (RES)
- no-connect marks 44 -> 51
Other:
- note added: "A1/A2 ~4gb microSD card goes in Teensy's port, NOT the Audio Adapter's. Keep microSD internal. Expose file transfer via a separate MTP mode. Don't write 64 individual files. Group them somehow for faster speeds. Transfer via MTP, as WAV format 2 APS6404L 8 MB PSRAM chips soldered on underside pads. Cut VBUS/GND or whatever"
- note added: "Bulk cap, near where power enters first LED, across +/- terminals Is this one polarized?"
- note added: "Center positive"
- note added: "Cue output from 3.5mm headphone jack?"
- note added: "FFC connectors/standoffs for connecting the 2 pcb's. Sending ~16 data pins to bottom pcb Ribbon cable needs to send multiple power/ground pins to distribute load (3/4) Consider high current from top board and noise"
- note added: "Likely will use U8g2 library instead of Adafruit 1306/GFX. SPI1 preferred so nothing weird happens with SPI0 (Audio Shield's SD/flash). If low on GPIO, can move it to SPI0 instead, should be fine. LOOK AT RESISTORS, CHECK TO SEE IT'S IN SPI MODE."
- note added: "Measure steady-state worst case amps and revisit the fuse only if needed. The current, higher PTC value means weaker protection against moderate overloads, but good for hard-faults. Use premade soft power switch board. Also allows for MCU-assisted shutdown procedure (save before shutdown)"
- note added: "Not sure how to implement kill/off, or if needed Cut VIN/VUSB, not sure which"
- note added: "Storage For 16-bit, total storage in Mb: (64 * Beats_per_loop * 10.584)/(BPM) For some DSP like pitch shift/tape-stop, converting to 32-bit float helps, but recording as 16-bit PCM is fine."
- note added: "Voltage rating 10/16v for comfort (for all caps, especially ones on 5v rail)"
- note added: "Wire1"
- note added: "Wire2"
- note removed: "APS6404L 8 MB PSRAM chip soldered on underside pads, between pins 31-32 and 33-34."
- note removed: "Bulk cap, near where power enters first LED, across +/- terminals"
- note removed: "Can move this I2C to Wire2, since we removed NeoKey"
- note removed: "microSD card goes in Teensy's port, NOT the Audio Adapter's."
- moved on the sheet: C1, C10, C11, C12, C13, C14, C15, C2, C3, C4, C5, C6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
