File: hardware/schematics/microloop.kicad_sch (KiCad schematic)
At the start: 75 parts, among them J1 Input L, J2 Output L, J3 Input R, J4 MIDI DIN-5, J5 Output R, J6 Barrel_Jack_Switch, J7 USB_C_Receptacle_USB2.0_14P, SW1 Rotary Encoder + Button, SW10 Preset Button, SW11 Preset Button, SW12 Preset Button, SW13 Preset Button, SW14 Preset Button, SW15 Preset Button, SW16 Preset Button, SW17 Preset Button, SW18 Preset Button, SW19 Preset Button, SW2 Rotary Encoder + Button, SW20 Preset Button, SW21 Preset Button, SW3 Rotary Encoder + Button, SW4 Rotary Encoder + Button, SW5 SW_Push, U1 Teensy 4.1, U2 Teensy Audio Shield (Rev D), U3 SSD1309 SPI OLED, U4 H11L1SM, U5 Encoders - MCP23017, U6 Adafruit 1400, U7 Switches - MCP23017, U8 SN74AHCT1G125

Commit message: decoupling caps
Parts:
- removed C10: 500uF, Capacitor_SMD:C_0805_2012Metric_Pad1.18x1.45mm_HandSolder, symbol Device:C
- removed C11, C12, C13, C14, C15, C8, C9: 0.1uF, Capacitor_SMD:C_0805_2012Metric_Pad1.18x1.45mm_HandSolder, symbol Device:C
- removed U5: Encoders - MCP23017, Package_SO:SOIC-28W_7.5x17.9mm_P1.27mm, symbol Interface_Expansion:MCP23017_SO
- removed U7: Switches - MCP23017, Package_SO:SOIC-28W_7.5x17.9mm_P1.27mm, symbol Interface_Expansion:MCP23017_SO
- added C20, C21, C22, C23, C24, C25, C26, C27, C28, C29, C30, C31, C32, C33: 0.1uF, symbol Device:C
- added R12, R13, R14, R15, R16, R17, R18, R19, R2, R20, R21, R22, R23, R24, R25, R26, R27, R28, R29, R3, R30, R31, R32, R33, R34, R35, R4, R5: 10kR, symbol Device:R_US
- added SW22, SW23, SW24: Menu Button, symbol Switch:SW_Push
- added SW6: Performance Encoder, symbol Device:RotaryEncoder_Switch
- added SW7, SW8: Menu Encoder, symbol Device:RotaryEncoder_Switch
- added U10: MCP23S17 #2, Package_SO:SOIC-28W_7.5x17.9mm_P1.27mm, symbol Interface_Expansion:MCP23S17_SO
- added U11: MCP23S17 #1, Package_SO:SOIC-28W_7.5x17.9mm_P1.27mm, symbol Interface_Expansion:MCP23S17_SO
- C1, C16, C2, C5, C7: footprint Capacitor_SMD:C_0805_2012Metric_Pad1.18x1.45mm_HandSolder -> (none)
- C18: value C_Polarized -> 680uF
- C3: value 0.1uF -> 1uF; footprint Capacitor_SMD:C_0805_2012Metric_Pad1.18x1.45mm_HandSolder -> (none)
- C4: value 0.1uF -> 10uF; footprint Capacitor_SMD:C_0805_2012Metric_Pad1.18x1.45mm_HandSolder -> (none)
- C6: value 0.1uF -> 47uF; footprint Capacitor_SMD:C_0805_2012Metric_Pad1.18x1.45mm_HandSolder -> (none)
- D10, D11, D12, D13, D14, D15, D16, D17, D18, D19, D8, D9: value SK6812MINI -> SK6812-E
- J6: value Barrel_Jack_Switch -> Barrel Jack
- R10: value 470R -> 4.7kR
- R11: value 330R/470R -> 330R
- SW1, SW2, SW3: value Rotary Encoder + Button -> Performance Encoder
- SW18, SW19, SW20, SW21: value Preset Button -> Effect Button
- SW4: value Rotary Encoder + Button -> Menu Encoder
- SW5: value SW_Push -> Power Button
Connections:
- net AA_3V is gone; now on net +3.3V: U1.46 (3V3), U2.28 (3V)
- net AA_SDCS is gone; now on net BEAT_LED: U1.12 (10_CS_MQSR), U2.12 (10_CS_MQSR)
- net ENC_A_1 is gone; now on net ENC_1_A: SW1.A
- net ENC_B_1 is gone; now on net ENC_1_B: SW1.B
- net ENC_B_2 is gone; now on net ENC_2_B: SW2.B
- net IOX_ENC_CLK is gone; now on net ENC_5_A: U1.38 (16_A2_RX4_SCL1), U2.20 (16_A2_RX4_SCL1)
- net IOX_ENC_SDA is gone; now on net ENC_4_B: U1.39 (17_A3_TX4_SDA1), U2.21 (17_A3_TX4_SDA1)
- net IOX_SW_CLK is gone; now on net ENC_2_A: U1.16 (24_A10_TX6_SCL2)
- net IOX_SW_INT is gone; now on net IND_LED_G: U1.20 (28_RX7)
- net IOX_SW_SDA is gone; now on net IND_LED_R: U1.17 (25_A11_RX6_SDA2)
- net +3.3V: now also C2.1, C3.1, C4.1, C5.1, C20.1, C33.1, R12.1, R13.1, R14.1, R15.1, R16.1, R17.1, R18.1, R19.1, R2.1, R20.1, R21.1, R22.1, R23.1, R24.1, R25.1, R26.1, R27.1, R28.1, R29.1, R3.1, R30.1, R31.1, R32.1, R33.1, R34.1, R35.1, R4.1, R5.1, U10.9 (VDD), U11.9 (VDD); no longer C16.1
- net +5V: now also C16.1, C18.1, U6.2 (OUT), C21.1, C22.1, C23.1, C24.1, C25.1, C26.1, C27.1, C28.1, C29.1, C30.1, C31.1, C32.1; no longer C2.1, C3.1, C4.1, C5.1
- net AA_MISO: no longer U1.14 (12_MISO_MQSL)
- net AA_MOSI: no longer U1.13 (11_MOSI_CTX1)
- net BEAT_LED: no longer U1.30 (38_CS1_IN1)
- net GND: now also C18.2, C20.2, C21.2, C22.2, C23.2, C24.2, C25.2, C26.2, C27.2, C28.2, C29.2, C30.2, C31.2, C32.2, C33.2, SW22.2, SW23.2, SW24.2, SW6.C, SW6.S2, SW7.C, SW7.S2, SW8.C, SW8.S2, U10.10 (VSS), U10.15 (A0), U10.16 (A1), U10.17 (A2), U11.10 (VSS), U11.15 (A0), U11.16 (A1), U11.17 (A2)
- net IND_LED_B: now also U1.21 (29_TX7); no longer U1.29 (37_CS)
- net IND_LED_G: no longer U1.28 (36_CS)
- net IND_LED_R: no longer U1.25 (33_MCLK2)
- net LINE_IN_DETECT: now also R18.2, U10.21 (GPA0); no longer U1.33 (41_A17)
- net LINE_OUT_DETECT: now also R19.2, U10.22 (GPA1); no longer U1.32 (40_A16)
- net OLED_CS: now also U2.2 (0_RX1_CRX2_CS1)
- net OLED_DC: now also U2.3 (1_TX1_CTX2_MISO1)
- net OLED_RES: now also U1.4 (2_OUT2), U2.4 (2_OUT2); no longer U1.44 (22_A8_CTX1), U2.26 (22_A8_CTX1)
- net PRST_SW_1: now also R5.2, U11.1 (GPB0); no longer U2.2 (0_RX1_CRX2_CS1)
- net PRST_SW_2: now also R20.2, U11.2 (GPB1); no longer U2.3 (1_TX1_CTX2_MISO1)
- net PRST_SW_3: now also R21.2, U11.3 (GPB2); no longer U2.4 (2_OUT2)
- net PRST_SW_4: now also R22.2, U11.4 (GPB3); no longer U2.5 (3_LRCLK2)
- net PRST_SW_5: now also R23.2, U11.5 (GPB4); no longer U2.6 (4_BCLK2)
- net PRST_SW_6: now also R24.2, U11.6 (GPB5); no longer U2.7 (5_IN2)
- net PRST_SW_7: now also R25.2, U11.7 (GPB6); no longer U2.11 (9_OUT1C)
- net PRST_SW_8: now also R26.2, U11.8 (GPB7)
- net ENC_1_B: now reaches U1.11 (9_OUT1C)
- net ENC_1_B: now also U2.11 (9_OUT1C)
- net ENC_2_B: now reaches U1.22 (30_CRX3)
- net ENC_3_A: now reaches U1.23 (31_CTX3)
- net ENC_3_A: now also SW6.A
- net ENC_3_B: now reaches U1.24 (32_OUT1B)
- net ENC_3_B: now also SW6.B
- net IOX_INT_1: now reaches U1.5 (3_LRCLK2)
- net IOX_INT_1: now also U2.5 (3_LRCLK2), U11.20 (INTA)
- net IOX_INT_2: now reaches U1.6 (4_BCLK2)
- net IOX_INT_2: now also U2.6 (4_BCLK2), U10.20 (INTA)
- net ENC_1_A: now reaches U1.7 (5_IN2)
- net ENC_1_A: now also U2.7 (5_IN2)
- net AA_MEMCS renamed AA_6
- net AA_SCK renamed IOX_SCK
- net IOX_SCK: now also U10.12 (SCK), U11.12 (SCK)
- net ENC_A_2 renamed ENC_2_A
- net ENC_A_3 renamed ENC_4_A
- net ENC_4_A: now also U1.44 (22_A8_CTX1), U2.26 (22_A8_CTX1)
- net ENC_A_4 renamed ENC_5_A
- net ENC_B_3 renamed ENC_4_B
- net ENC_B_4 renamed ENC_5_B
- net ENC_5_B: now also U1.33 (41_A17)
- net ENC_SW_1 renamed ENC_1_SW
- net ENC_1_SW: now also R2.2, U10.1 (GPB0)
- net ENC_SW_2 renamed ENC_2_SW
- net ENC_2_SW: now also R17.2, U10.2 (GPB1)
- net ENC_SW_3 renamed ENC_4_SW
- net ENC_4_SW: now also R15.2, U10.4 (GPB3)
- net ENC_SW_4 renamed ENC_5_SW
- net ENC_5_SW: now also R12.2, U10.5 (GPB4)
- net IOX_ENC_INT renamed ENC_6_B
- net ENC_6_B: now also SW7.B
- net PRST_SW_10 renamed EFCT_SW_2
- net EFCT_SW_2: now also R28.2, U11.22 (GPA1)
- net PRST_SW_11 renamed EFCT_SW_3
- net EFCT_SW_3: now also R29.2, U11.23 (GPA2)
- net PRST_SW_12 renamed EFCT_SW_4
- net EFCT_SW_4: now also R30.2, U11.24 (GPA3)
- net PRST_SW_9 renamed EFCT_SW_1
- net EFCT_SW_1: now also R27.2, U11.21 (GPA0)
- new net: R34.2, U11.18 (~{RESET})
- new net: R4.2, U10.18 (~{RESET})
- new net ENC_3_SW: R16.2, SW6.S1, U10.3 (GPB2)
- new net ENC_6_A: SW7.A, U1.32 (40_A16)
- new net ENC_6_SW: R13.2, SW7.S1, U10.6 (GPB5)
- new net ENC_7_A: SW8.A, U1.30 (38_CS1_IN1)
- new net ENC_7_B: SW8.B, U1.25 (33_MCLK2)
- new net ENC_7_SW: R14.2, SW8.S1, U10.7 (GPB6)
- new net IOX_CS_1: R35.2, U1.28 (36_CS), U11.11 (~{CS})
- new net IOX_CS_2: R3.2, U1.29 (37_CS), U10.11 (~{CS})
- new net IOX_MISO: U1.14 (12_MISO_MQSL), U10.14 (SO), U11.14 (SO)
- new net IOX_MOSI: U1.13 (11_MOSI_CTX1), U10.13 (SI), U11.13 (SI)
- new net MENU_SW_1: R31.2, SW22.1, U11.25 (GPA4)
- new net MENU_SW_2: R32.2, SW23.1, U11.26 (GPA5)
- new net MENU_SW_3: R33.2, SW24.1, U11.27 (GPA6)
Other:
- note added: "A1/A2 ~4gb microSD card goes in Teensy's port, NOT the Audio Adapter's. Keep microSD internal. Expose file transfer via a separate MTP mode. Don't write 64 individual files. Group them somehow for faster speeds. Transfer via MTP, as WAV format 2 APS6404L 8 MB PSRAM chips soldered on underside pads. Cut VIN/VUSB MAKE SURE that total 3.3v output DOESN'T EXCEED 250mA"
- note added: "Disable internal pull-ups in software. Use active-low, push-pull interrupts."
- note added: "TOP-BOARD FFC ENTRY Add rail entry caps"
- note added: "Using optional SD card/MEM chip pins. Make sure to free them if using in the future."
- note removed: "A1/A2 ~4gb microSD card goes in Teensy's port, NOT the Audio Adapter's. Keep microSD internal. Expose file transfer via a separate MTP mode. Don't write 64 individual files. Group them somehow for faster speeds. Transfer via MTP, as WAV format 2 APS6404L 8 MB PSRAM chips soldered on underside pads. Cut VBUS/GND or whatever"
- note removed: "Bulk cap, near where power enters first LED, across +/- terminals Is this one polarized?"
- note removed: "Place decoupling capacitor as close as possible to MCP23017 VDD and VSS pins."
- note removed: "Place decoupling capacitors as close as possible from VDD/VSS or VCC/GND"
- note removed: "Wire1"
- note removed: "Wire2"
- moved on the sheet: C17, C18, C19, D1, D10, D11, D12, D13, D14, D15, D16, D17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

Commit message: usb-c schematic
Parts:
- removed C17: 47uF, symbol Device:C_Polarized
- removed C19: 0.1uF, Capacitor_SMD:C_0805_2012Metric_Pad1.18x1.45mm_HandSolder, symbol Device:C
- added C10, C8, C9: 47uF, symbol Device:C_Polarized
- added C34, C35, C37: 0.1uF, symbol Device:C
- added C36: 1uF, symbol Device:C
- added D5: ESDA051-1JY TVS, symbol Device:D_Zener
- added R38: 0R, symbol Device:R_US
- added R42, R43: 5.1kR, symbol Device:R_US
- added U5: TPD6S300ARUKR, WQFN20_RUK_TEX, symbol TPD6S300ARUKR:TPD6S300ARUKR
- C6: value 47uF -> 2.2uF
- D3: value D_TVS -> SMBJ6.0CA TVS
- F1: value Polyfuse -> PTC Polyfuse
- J7: value USB_C_Receptacle_USB2.0_14P -> USB-C Receptacle
Connections:
- net +3.3V: now also C36.2, U5.10 (VPWER)
- net +5V: now also C10.1, C34.1, C8.1; no longer C6.1
- net GND: now also J7.A1 (GND), J7.A12 (GND), J7.B1 (GND), J7.B12 (GND), C10.2, C34.2, C35.2, C36.1, C37.1, C8.2, C9.2, D5.2 (A), R38.2, R42.2, R43.2, U5.13 (GND), U5.16 (NC), U5.17 (NC), U5.18 (GND), U5.21 (GND), U5.6 (RPD_G2), U5.7 (RPD_G1), U5.8 (GND)
- net at D3.1 (A1), F1.2, U6.1 (IN): now also C35.1, C9.1
- net USB_VBUS: now reaches J7.A4 (VBUS), J7.A9 (VBUS), J7.B4 (VBUS), J7.B9 (VBUS)
- net USB_VBUS: now also C6.1, U1.49 (VUSB), D5.1 (K)
- net USB_CC1: now reaches J7.A5 (CC1)
- net USB_CC1: now also U5.4 (C_CC1)
- net USB_D+: now reaches J7.A6 (D+)
- net USB_D+: now also J7.B6 (D+), U5.1 (C_SBU1), U5.20 (D1)
- net USB_D-: now reaches J7.A7 (D-)
- net USB_D-: now also J7.B7 (D-), U5.19 (D2), U5.2 (C_SBU2)
- net USB_CC2: now reaches J7.B5 (CC2)
- net USB_CC2: now also U5.5 (C_CC2)
- net at J7.S1 (SHIELD): now also R38.1
- net USB_OUT_D-: now reaches U1.66 (D-)
- net USB_OUT_D-: now also U5.14 (SBU2)
- net USB_OUT_D+: now reaches U1.67 (D+)
- net USB_OUT_D+: now also U5.15 (SBU1)
- new net: C37.2, U5.3 (VBIAS)
- new net: R43.1, U5.12 (CC1)
- new net: R42.1, U5.11 (CC2)
- no-connect marks 51 -> 49
Other:
- note added: "In footprint: VBUS is A4, A9, B4, B9 tied together GND is A1, A12, B1, B12 tied together TVS to GND should be THE SHORTEST"
- note added: "Keep lines between Audio shield and jacks as SHORT AS POSSIBLE"
- note added: "Make sure to add header through holes in PCB to connect Line In/Out/GND to PCB Using optional SD card/MEM chip pins. Make sure to free them if using in the future."
- note added: "Pin 3 cap NEEDS to be rated 50V for headroom Pin 21 is the exposed middle pad"
- note added: "Single point connection to GND, just in case later one I want a real metal chassis ground for EMI/other reasons."
- note removed: "Using optional SD card/MEM chip pins. Make sure to free them if using in the future."
- moved on the sheet: C2, C4, C5, C7, D3, D7, F1, J4, J6, J7, R10, R9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

Commit message: backups
Parts:
- removed SW1, SW2, SW3, SW6: Performance Encoder, symbol Device:RotaryEncoder_Switch
- removed SW4, SW7, SW8: Menu Encoder, symbol Device:RotaryEncoder_Switch
- added C39, C40, C41, C42, C43, C44, C45, C46, C47, C48, C49, C50, C51, C52: 0.01uF, symbol Device:C
- added R39, R40, R41, R44, R45, R46, R47, R48, R49, R50, R51, R52, R53, R54, R55, R56, R57, R58, R59, R60, R61, R62, R63, R64, R65, R66, R67, R68: 10kR, symbol Device:R_US
- added SW25, SW26, SW27, SW28: Performance Encoder, symbol Device:RotaryEncoder_Switch
- added SW29, SW30, SW31: Menu Encoder, symbol Device:RotaryEncoder_Switch
Connections:
- net +3.3V: now also R40.1, R41.1, R45.1, R47.1, R49.1, R51.1, R53.1, R55.1, R57.1, R59.1, R61.1, R63.1, R65.1, R67.1
- net ENC_1_A: now also R39.1, R40.2
- net ENC_1_B: now also R41.2, R44.1
- net ENC_1_SW: now also SW25.S1
- net ENC_2_A: now also R47.2, R48.1
- net ENC_2_B: now also R45.2, R46.1
- net ENC_2_SW: now also SW26.S1
- net ENC_3_A: now also R51.2, R52.1
- net ENC_3_B: now also R49.2, R50.1
- net ENC_3_SW: now also SW27.S1
- net ENC_4_A: now also R55.2, R56.1
- net ENC_4_B: now also R53.2, R54.1
- net ENC_4_SW: now also SW28.S1
- net ENC_5_A: now also R59.2, R60.1
- net ENC_5_B: now also R57.2, R58.1
- net ENC_5_SW: now also SW29.S1
- net ENC_6_A: now also R63.2, R64.1
- net ENC_6_B: now also R61.2, R62.1
- net ENC_6_SW: now also SW30.S1
- net ENC_7_A: now also R67.2, R68.1
- net ENC_7_B: now also R65.2, R66.1
- net ENC_7_SW: now also SW31.S1
- net GND: now also C39.2, C40.2, C41.2, C42.2, C43.2, C44.2, C45.2, C46.2, C47.2, C48.2, C49.2, C50.2, C51.2, C52.2, SW25.C, SW25.S2, SW26.C, SW26.S2, SW27.C, SW27.S2, SW28.C, SW28.S2, SW29.C, SW29.S2, SW30.C, SW30.S2, SW31.C, SW31.S2
- new net: C40.1, R44.2, SW25.B
- new net: C48.1, R60.2, SW29.A
- new net: C50.1, R64.2, SW30.A
- new net: C49.1, R62.2, SW30.B
- new net: C52.1, R68.2, SW31.A
- new net: C41.1, R46.2, SW26.B
- new net: C42.1, R48.2, SW26.A
- new net: C39.1, R39.2, SW25.A
- new net: C46.1, R56.2, SW28.A
- new net: C43.1, R50.2, SW27.B
- new net: C45.1, R54.2, SW28.B
- new net: C47.1, R58.2, SW29.B
- new net: C44.1, R52.2, SW27.A
- new net: C51.1, R66.2, SW31.B
Other:
- note added: "2x24 FFC connectors 1 for fast/direct lines: encoders + dome leds 1 for bus/control/power: SPI's, SN74"
- note added: "FFC1 - fast/direct lines Use this for the stuff you want most isolated and straightforward: 7 encoders + 4 dome LED lines, with grounds sprinkled in. GND ENC1_A ENC1_B GND ENC2_A ENC2_B GND ENC3_A ENC3_B GND ENC4_A ENC4_B GND ENC5_A ENC5_B LED_BEAT ENC6_A ENC6_B GND ENC7_A ENC7_B LED_RGB_R LED_RGB_G LED_RGB_B That gives you 18 direct signal lines + 6 grounds = 24 pins."
- note added: "FFC2 - bus/control/power Use this for the two SPI buses, interrupts, LED-data, and the rails. 5V GND 5V GND 3V3 GND OLED_SCK OLED_MOSI OLED_CS OLED_DC OLED_RES GND IO_SCK IO_MOSI IO_MISO IO_CS1 IO_CS2 IO_INT1 IO_INT2 GND LED_DATA_BUF GND SPARE / RESET / FUTURE_GPIO GND That gives you: 13 signal lines 2× 5V 1× 3V3 7 grounds 1 spare"
- note added: "Put filters closer to teensy (bottom pcb?) Use a proper quadrature state-table decoder in firmware, not a naive "edge on A, read B" approach."
- note removed: "TOP-BOARD FFC ENTRY Add rail entry caps"
- moved on the sheet: C1, C20, C3, R12, R13, R14, R15, R16, R17, R18, R19, R2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
